File: pcb/imu.kicad_sch (KiCad schematic)
At the start: 12 parts, among them U16 BNO055, Y1 Crystal_GND24

Commit message: Add new IMU revision and more info in readme
Parts:
- added C22, C24, C25, C26?, C29, C36, C98, C99, C?: C, symbol Device:C
- added Q30, Q31: NMOS, symbol Simulation_SPICE:NMOS
- added R137, R?: 4K7, symbol Device:R
- added R144, R?: 0, symbol Device:R
- added R64, R66: 10K, symbol Device:R
- added U16: BHI260AP, BHI260AP, symbol BHI260AP:BHI260AP
- added U38: BMM150, BMM150, symbol BMM150:BMM150
- added U39: W25Q64JWSSIQ, SOIC127P790X216-8N, symbol W25Q64JWSSIQ:W25Q64JWSSIQ
- added U40: MCP1700x-180xxTT, Package_TO_SOT_SMD:SOT-23, symbol Regulator_Linear:MCP1700x-180xxTT
Connections:
- net GND: now also C22.2, C24.2, C25.2, C26?.2, C29.2, C36.2, C98.2, C99.2, C?.1, R144.1, U16.17 (GNDIO_1), U16.25 (GND_1), U16.26 (GND_2), U16.27 (GND_3), U16.32 (HSDO), U16.36 (GNDIO_2), U38.A5 (CSB), U38.C1 (SDO), U38.C5 (GND_1), U38.E1 (GND_2), U38.E3 (GND_3), U39.4 (GND), U40.1 (GND)
- net PB2_I2C0SCL: now also Q30.1 (D)
- net PB3_I2C0SDA: now also Q31.1 (D)
- net VCC: now also C22.1, U40.3 (VI)
- new net: C24.1, C25.1, C26?.1, C29.1, C36.1, C98.1, C99.1, Q30.2 (G), Q31.2 (G), R137.2, R64.1, R66.1, R?.1, R?.2, U16.12 (VDDIO_2), U16.28 (VDD), U16.42 (VDDIO_3), U16.7 (VDDIO_1), U16.9 (RESETN), U38.A1 (PS), U38.B2 (VDDIO), U38.E5 (VDD), U39.8 (VCC), U40.2 (VO)
- new net: Q30.3 (S), R66.2, U16.33 (HSCX)
- new net: Q31.3 (S), R64.2, U16.11 (HSDX)
- new net: U16.14 (QSPI_CSN), U39.1 (~{CS})
- new net: U16.15 (QSPI_D1), U39.2 (DO_(IO1))
- new net: U16.18 (MCSB2), U38.D2 (INT), U38.D4 (DRDY)
- new net: U16.20 (QSPI_D2), U39.7 (~{HOLD_OR_}/RESET_(IO3))
- new net: R?.1, U16.22 (ASCX), U38.A3 (SCK)
- new net: R144.2, U16.3 (HOSTBOOT)
- new net: R137.1, U16.30 (ASDX), U38.B4 (SDI)
- new net: R?.2, U16.34 (HCSB)
- new net: U16.4 (QSPI_D0), U39.5 (DI_(IO0))
- new net: U16.5 (QSPI_CLK), U39.6 (CLK)
- new net: C?.2, U16.6 (VREG)
- new net: U16.8 (QSPI_D3), U39.3 (~{WP_(IO2)})
- no-connect marks 2 -> 21
Other:
- note added: "Revision <= 2.3"
- note added: "Revision > 2.3 IMU"
- moved on the sheet: C22, C24, C25, C26, C29, C36, R64, R65, R66, R68, U16, Y1
