File: pcb/usb.kicad_sch (KiCad schematic)
At the start: 31 parts, among them J17 USB_B_Mini, Q22 PMOS, Q23 PMOS, Q25 NMOS, Q27 PMOS, U15 FT230XQ, U19 PUSBM5V5X4-TL_115

Commit message: Add new IMU revision and more info in readme
Other:
- note added: "L2 is an educated guess"
Changed lines of the file:
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@@
+		)
+	)
+	(text "L2 is an educated guess"
+		(exclude_from_sim no)
+		(at 163.83 124.46 0)
+		(effects
+			(font
+				(size 1.27 1.27)
+			)
 		)
 	)
