File: pcb/encoder.kicad_sch (KiCad schematic)
At the start: 3 parts, among them J22 Conn_01x04_Pin, U35 CPDV5-3V3UP

Commit message: Update motor encoder TVS diodes to be the correct voltage
Parts:
- U35: value CPDV5-3V3UP -> CPDV5-5V0U; symbol CPDV5:CPDV5-3V3UP -> CPDV5:CPDV5-5V0U
Changed lines of the file:
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@@
 	)
 	(symbol
-		(lib_id "CPDV5:CPDV5-3V3UP")
+		(lib_id "CPDV5:CPDV5-5V0U")
 		(at 120.65 93.98 0)
 		(unit 1)
@@
 			)
 		)
-		(property "Value" "CPDV5-3V3UP"
+		(property "Value" "CPDV5-5V0U"
 			(at 135.89 88.9 0)
 			(show_name no)
@@
 			)
 		)
-		(property "Datasheet" "CPDV5-3V3UP"
+		(property "Datasheet" "CPDV5-5V0U"
 			(at 120.65 93.98 0)
 			(hide yes)
